Commit message: robot state publisher added to highlevel interface docker

File: deploy/ros2_ws/src/b1_description/robots/robot_virtual_arm.xacro (robot description, xacro)
@@ -13,8 +13,8 @@
             <origin rpy="0 0 0" xyz="0 0 0"/>
             <parent link="world"/>
-            <child link="base"/>
+            <child link="base_link"/>
         </joint>
     </xacro:if>
-    <link name="base">
+    <link name="base_link">
         <visual>
             <origin rpy="0 0 0" xyz="0 0 0"/>
@@ -26,5 +26,5 @@
     <joint name="floating_base" type="fixed">
         <origin rpy="0 0 0" xyz="0 0 0"/>
-        <parent link="base"/>
+        <parent link="base_link"/>
         <child link="trunk"/>
     </joint>
@@ -83,17 +83,4 @@
         </collision>
     </link>
-    <link name="b1_rslidar">
-        <visual>
-            <origin rpy="0 0 0" xyz="0 0 0"/>
-            <geometry>
-                <box size="0.2 0.2 0.2"/>
-            </geometry>
-        </visual>
-    </link>
-    <joint name="lidar_joint" type="fixed">
-        <parent link="imu_link"/>
-        <child link="b1_rslidar"/>
-        <origin rpy="0 0 0" xyz="0.2 0 0.3"/>
-    </joint>
     <link name="virtual_arm">
         <visual>
