Commit message: IMU to trunk extrinsics are corrected

File: deploy/ros2_ws/src/b1_description/robots/robot.xacro (robot description, xacro)
@@ -61,5 +61,5 @@
         <parent link="trunk"/>
         <child link="imu_link"/>
-        <origin rpy="0 0 0" xyz="0 0 0"/>
+        <origin rpy="0 0 0.015" xyz="-0.024 0 0.07"/>
     </joint>
     <link name="imu_link">

File: deploy/ros2_ws/src/b1_description/robots/robot_virtual_arm.xacro (robot description, xacro)
@@ -61,5 +61,5 @@
         <parent link="trunk"/>
         <child link="imu_link"/>
-        <origin rpy="0 0 0" xyz="0 0 0"/>
+        <origin rpy="0 0 0.015" xyz="-0.024 0 0.07"/>
     </joint>
     <link name="imu_link">
